File: Hardware/Frame/espglasses/snapshots/espglasses_snapshot_step3_pcb_layout_started_20260324_120950/espglasses.kicad_pcb (KiCad board)
At the start: 2 copper layers, 170 x 45 mm, 13 parts, among them J1 BATTERY_1S, J2 OLED_SH1106_I2C, J3 TOUCH_INPUTS, J4 AUDIO_OUT_MONO, J5 UART_BOOT_DEBUG, J6 LED_STATUS, U1 ESP32_DEV_BOARD_PIN_BREAKOUT

Commit message: kicad checkpoint
Connections:
- C1 pad 1: +3V3_DIG -> (no net)
- C1 pad 2: GND -> (no net)
- C2 pad 1: +3V3_DIG -> (no net)
- C2 pad 2: GND -> (no net)
- D1 pad 1: GND -> (no net)
- D1 pad 2: LED_A -> (no net)
- J1 pad 1: VBAT_RAW -> (no net)
- J1 pad 2: GND -> (no net)
- J2 pad 1: +3V3_DIG -> (no net)
- J2 pad 2: GND -> (no net)
- J2 pad 3: I2C_SCL -> (no net)
- J2 pad 4: I2C_SDA -> (no net)
- J3 pad 1: TOUCH1_IN -> (no net)
- J3 pad 2: TOUCH2_IN -> (no net)
- J4 pad 1: DAC_SUM -> (no net)
- J4 pad 2: GND -> (no net)
- J5 pad 1: UART_TX_DBG -> (no net)
- J5 pad 2: UART_RX_DBG -> (no net)
- J5 pad 3: EN -> (no net)
- J5 pad 4: IO0 -> (no net)
- J5 pad 5: +3V3_DIG -> (no net)
- J5 pad 6: GND -> (no net)
- J6 pad 1: LED_STAT -> (no net)
- J6 pad 2: GND -> (no net)
- R1 pad 1: LED_STAT -> (no net)
- R1 pad 2: LED_A -> (no net)
- R2 pad 1: DAC_L_OUT -> (no net)
- R2 pad 2: DAC_SUM -> (no net)
- R3 pad 1: DAC_R_OUT -> (no net)
- R3 pad 2: DAC_SUM -> (no net)
- U1 pad 1: GND -> (no net)
- U1 pad 10: UART_TX_DBG -> (no net)
- U1 pad 12: UART_RX_DBG -> (no net)
- U1 pad 14: DAC_R_OUT -> (no net)
- U1 pad 16: DAC_L_OUT -> (no net)
- U1 pad 2: +3V3_DIG -> (no net)
- U1 pad 24: TOUCH2_IN -> (no net)
- U1 pad 26: TOUCH1_IN -> (no net)
- U1 pad 32: I2C_SCL -> (no net)
- U1 pad 34: I2C_SDA -> (no net)
- U1 pad 4: IO0 -> (no net)
- U1 pad 6: EN -> (no net)
- U1 pad 8: LED_STAT -> (no net)
Changed lines of the file:
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@@
 	)
 	(net 0 "")
-	(net 1 "UART_RX_DBG")
-	(net 2 "I2C_SDA")
-	(net 3 "VBAT_RAW")
-	(net 4 "GND")
-	(net 5 "I2C_SCL")
-	(net 6 "LED_A")
-	(net 7 "IO0")
-	(net 8 "EN")
-	(net 9 "+3V3_DIG")
-	(net 10 "TOUCH2_IN")
-	(net 11 "TOUCH1_IN")
-	(net 12 "DAC_SUM")
-	(net 13 "DAC_R_OUT")
-	(net 14 "UART_TX_DBG")
-	(net 15 "LED_STAT")
-	(net 16 "DAC_L_OUT")
 	(footprint "LED_0603_1608Metric"
 		(layer "F.Cu")
@@
 			(layers "F.Cu" "F.Mask" "F.Paste")
 			(roundrect_rratio 0.25)
-			(net 4 "GND")
 		)
 		(pad "2" smd roundrect
@@
 			(layers "F.Cu" "F.Mask" "F.Paste")
 			(roundrect_rratio 0.25)
-			(net 6 "LED_A")
 		)
 		(embedded_fonts no)
@@
 			(layers "*.Cu" "*.Mask")
 			(remove_unused_layers no)
-			(net 9 "+3V3_DIG")
 		)
 		(pad "2" thru_hole circle
@@
 			(layers "*.Cu" "*.Mask")
 			(remove_unused_layers no)
-			(net 4 "GND")
 		)
 		(pad "3" thru_hole circle
@@
 			(layers "*.Cu" "*.Mask")
 			(remove_unused_layers no)
-			(net 5 "I2C_SCL")
 		)
 		(pad "4" thru_hole circle
@@
 			(layers "*.Cu" "*.Mask")
 			(remove_unused_layers no)
-			(net 2 "I2C_SDA")
 		)
 		(embedded_fonts no)
@@
 			(layers "F.Cu" "F.Mask" "F.Paste")
 			(roundrect_rratio 0.25)
-			(net 16 "DAC_L_OUT")
 		)
 		(pad "2" smd roundrect
@@
 			(layers "F.Cu" "F.Mask" "F.Paste")
 			(roundrect_rratio 0.25)
-			(net 12 "DAC_SUM")
 		)
 		(embedded_fonts no)
@@
 			(layers "*.Cu" "*.Mask")
 			(remove_unused_layers no)
-			(net 12 "DAC_SUM")
 		)
 		(pad "2" thru_hole circle
@@
 			(layers "*.Cu" "*.Mask")
 			(remove_unused_layers no)
-			(net 4 "GND")
 		)
 		(embedded_fonts no)
@@
 			(layers "F.Cu" "F.Mask" "F.Paste")
 			(roundrect_rratio 0.25)
-			(net 9 "+3V3_DIG")
 		)
 		(pad "2" smd roundrect
@@
 			(layers "F.Cu" "F.Mask" "F.Paste")
 			(roundrect_rratio 0.25)
-			(net 4 "GND")
 		)
 		(embedded_fonts no)
@@
 			(layers "F.Cu" "F.Mask" "F.Paste")
 			(roundrect_rratio 0.25)
-			(net 15 "LED_STAT")
 		)
 		(pad "2" smd roundrect
@@
 			(layers "F.Cu" "F.Mask" "F.Paste")
 			(roundrect_rratio 0.25)
-			(net 6 "LED_A")
 		)
 		(embedded_fonts no)
@@
 			(layers "F.Cu" "F.Mask" "F.Paste")
 			(roundrect_rratio 0.25)
-			(net 13 "DAC_R_OUT")
 		)
 		(pad "2" smd roundrect
@@
 			(layers "F.Cu" "F.Mask" "F.Paste")
 			(roundrect_rratio 0.25)
-			(net 12 "DAC_SUM")
 		)
 		(embedded_fonts no)
@@
 			(remove_unused_layers no)
 			(roundrect_rratio 0.208333)
-			(net 3 "VBAT_RAW")
 		)
 		(pad "2" thru_hole oval
@@
 			(layers "*.Cu" "*.Mask")
 			(remove_unused_layers no)
-			(net 4 "GND")
 		)
 		(embedded_fonts no)
@@
 			(layers "F.Cu" "F.Mask" "F.Paste")
 			(roundrect_rratio 0.25)
-			(net 9 "+3V3_DIG")
 		)
 		(pad "2" smd roundrect
@@
 			(layers "F.Cu" "F.Mask" "F.Paste")
 			(roundrect_rratio 0.25)
-			(net 4 "GND")
 		)
 		(embedded_fonts no)
@@
 			(layers "*.Cu" "*.Mask")
 			(remove_unused_layers no)
-			(net 11 "TOUCH1_IN")
 		)
 		(pad "2" thru_hole circle
@@
 			(layers "*.Cu" "*.Mask")
 			(remove_unused_layers no)
-			(net 10 "TOUCH2_IN")
 		)
 		(embedded_fonts no)
@@
 			(layers "*.Cu" "*.Mask")
 			(remove_unused_layers no)
-			(net 14 "UART_TX_DBG")
 		)
 		(pad "2" thru_hole circle
@@
 			(layers "*.Cu" "*.Mask")
 			(remove_unused_layers no)
-			(net 1 "UART_RX_DBG")
 		)
 		(pad "3" thru_hole circle
@@
 			(layers "*.Cu" "*.Mask")
 			(remove_unused_layers no)
-			(net 8 "EN")
 		)
 		(pad "4" thru_hole circle
@@
 			(layers "*.Cu" "*.Mask")
 			(remove_unused_layers no)
-			(net 7 "IO0")
 		)
 		(pad "5" thru_hole circle
@@
 			(layers "*.Cu" "*.Mask")
 			(remove_unused_layers no)
-			(net 9 "+3V3_DIG")
 		)
 		(pad "6" thru_hole circle
@@
 			(layers "*.Cu" "*.Mask")
 			(remove_unused_layers no)
-			(net 4 "GND")
 		)
 		(embedded_fonts no)
@@
 			(size 1.5 0.9)
 			(layers "F.Cu" "F.Mask" "F.Paste")
-			(net 4 "GND")
 		)
 		(pad "2" smd rect
@@
 			(size 1.5 0.9)
 			(layers "F.Cu" "F.Mask" "F.Paste")
-			(net 9 "+3V3_DIG")
 		)
 		(pad "3" smd rect
@@
 			(size 1.5 0.9)
 			(layers "F.Cu" "F.Mask" "F.Paste")
-			(net 7 "IO0")
 		)
 		(pad "5" smd rect
@@
 			(size 1.5 0.9)
 			(layers "F.Cu" "F.Mask" "F.Paste")
-			(net 8 "EN")
 		)
 		(pad "7" smd rect
@@
 			(size 1.5 0.9)
 			(layers "F.Cu" "F.Mask" "F.Paste")
-			(net 15 "LED_STAT")
 		)
 		(pad "9" smd rect
@@
 			(size 1.5 0.9)
 			(layers "F.Cu" "F.Mask" "F.Paste")
-			(net 14 "UART_TX_DBG")
 		)
 		(pad "11" smd rect
@@
 			(size 1.5 0.9)
 			(layers "F.Cu" "F.Mask" "F.Paste")
-			(net 1 "UART_RX_DBG")
 		)
 		(pad "13" smd rect
@@
 			(size 1.5 0.9)
 			(layers "F.Cu" "F.Mask" "F.Paste")
-			(net 13 "DAC_R_OUT")
 		)
 		(pad "15" smd rect
@@
 			(size 1.5 0.9)
 			(layers "F.Cu" "F.Mask" "F.Paste")
-			(net 16 "DAC_L_OUT")
 		)
 		(pad "17" smd rect
@@
 			(size 1.5 0.9)
 			(layers "F.Cu" "F.Mask" "F.Paste")
-			(net 10 "TOUCH2_IN")
 		)
 		(pad "25" smd rect
@@
 			(size 1.5 0.9)
 			(layers "F.Cu" "F.Mask" "F.Paste")
-			(net 11 "TOUCH1_IN")
 		)
 		(pad "27" smd rect
@@
 			(size 1.5 0.9)
 			(layers "F.Cu" "F.Mask" "F.Paste")
-			(net 5 "I2C_SCL")
 		)
 		(pad "33" smd rect
@@
 			(size 1.5 0.9)
 			(layers "F.Cu" "F.Mask" "F.Paste")
-			(net 2 "I2C_SDA")
 		)
 		(pad "35" smd rect
@@
 			(layers "*.Cu" "*.Mask")
 			(remove_unused_layers no)
-			(net 15 "LED_STAT")
 		)
 		(pad "2" thru_hole circle
@@
 			(layers "*.Cu" "*.Mask")
 			(remove_unused_layers no)
-			(net 4 "GND")
 		)
 		(embedded_fonts no)
@@
 		)
 	)
-	(gr_rect
-		(start 0 0)
+	(gr_line
+		(start 170 45)
+		(end 0 45)
+		(stroke
+			(width 0.1)
+			(type default)
+		)
+		(layer "Edge.Cuts")
+	)
+	(gr_line
+		(start 0 45)
+		(end 0 0)
+		(stroke
+			(width 0.1)
+			(type default)
+		)
+		(layer "Edge.Cuts")
+	)
+	(gr_line
+		(start 170 0)
 		(end 170 45)
 		(stroke
@@
 			(type default)
 		)
-		(fill no)
 		(layer "Edge.Cuts")
 	)
+	(gr_line
+		(start 0 0)
+		(end 170 0)
+		(stroke
+			(width 0.1)
+			(type default)
+		)
+		(layer "Edge.Cuts")
+	)
