File: Hardware/Frame/espglasses/espglasses.kicad_sch (KiCad schematic)
At the start: 0 parts

Commit message: kicad start
Parts:
- added C1: 10uF, symbol Device:C
- added C2: 100nF, symbol Device:C
- added D1: GREEN, symbol Device:LED
- added J1: BATTERY_1S, symbol Connector_Generic:Conn_01x02
- added J2: OLED_SH1106_I2C, symbol Connector_Generic:Conn_01x04
- added J3: TOUCH_INPUTS, symbol Connector_Generic:Conn_01x02
- added J4: AUDIO_OUT_MONO, symbol Connector_Generic:Conn_01x02
- added J5: UART_BOOT_DEBUG, symbol Connector_Generic:Conn_01x06
- added J6: LED_STATUS, symbol Connector_Generic:Conn_01x02
- added R1: 1k, symbol Device:R
- added R2, R3: 10k, symbol Device:R
- added U1: ESP32_DEV_BOARD_PIN_BREAKOUT, symbol Connector_Generic:Conn_02x19_Odd_Even
- added _TEMPLATE_C: C_TEMPLATE, symbol Device:C
- added _TEMPLATE_D: LED_TEMPLATE, symbol Device:LED
- added _TEMPLATE_R: R_TEMPLATE, symbol Device:R
Changed lines of the file:
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@@
-(kicad_sch
-	(version 20250114)
-	(generator "eeschema")
-	(generator_version "9.0")
-	(paper "A4")
-	(sheet_instances
-		(path "/"
-			(page "1")
-		)
-	)
-	(embedded_fonts no)
-)

Commit message: kicad checkpoint
Parts:
- removed J4: AUDIO_OUT_MONO, symbol Connector_Generic:Conn_01x02
- removed J6: LED_STATUS, symbol Connector_Generic:Conn_01x02
- added C3: 10uF, Capacitor_SMD:C_0603_1608Metric, symbol Device:C
- added C4, C5: 100nF, Capacitor_SMD:C_0603_1608Metric, symbol Device:C
- added J4: UART_BOOT_DEBUG, Connector_PinHeader_2.54mm:PinHeader_1x06_P2.54mm_Vertical, symbol Connector_Generic:Conn_01x06
- added R4, R5: 10k, Resistor_SMD:R_0603_1608Metric, symbol Device:R
- added U2: OV2640_CAMERA_IF, Connector_FFC-FPC:TE_1734839-0_1x20-1MP_P0.5mm_Horizontal, symbol Connector_Generic:Conn_02x10_Odd_Even
- added U3: MPU6050_CORE, Package_QFN:QFN-24-1EP_4x4mm_P0.5mm_EP2.6x2.6mm, symbol Connector_Generic:Conn_01x08
- added U4: INMP441_CORE, Package_LGA:LGA-6_3x4mm_P0.5mm, symbol Connector_Generic:Conn_01x06
- added U5: LIION_CHARGER_IC_CORE, Package_SO:SOIC-8_3.9x4.9mm_P1.27mm, symbol Connector_Generic:Conn_01x08
- added U6: REGULATOR_3V3_CORE, Package_TO_SOT_SMD:SOT-223-3_TabPin2, symbol Connector_Generic:Conn_01x05
- added U7: AUDIO_AMP_CORE, Package_SO:SOIC-16_3.9x9.9mm_P1.27mm, symbol Connector_Generic:Conn_01x08
- C1, C2: footprint (none) -> Capacitor_SMD:C_0603_1608Metric
- D1: footprint (none) -> LED_SMD:LED_0603_1608Metric
- J1: footprint (none) -> Connector_JST:JST_PH_B2B-PH-K_1x02_P2.00mm_Vertical
- J2: value OLED_SH1106_I2C -> OLED_I2C_PANEL; footprint (none) -> Connector_PinHeader_2.54mm:PinHeader_1x04_P2.54mm_Vertical
- J3: value TOUCH_INPUTS -> SPEAKER_8OHM; footprint (none) -> Connector_PinHeader_2.54mm:PinHeader_1x02_P2.54mm_Vertical
- J5: value UART_BOOT_DEBUG -> USBC_POWER_IN; footprint (none) -> Connector_USB:USB_C_Receptacle_HRO_TYPE-C-31-M-12
- R1, R2, R3: footprint (none) -> Resistor_SMD:R_0603_1608Metric
- U1: value ESP32_DEV_BOARD_PIN_BREAKOUT -> ESP32_WROVER_E_CORE; footprint (none) -> RF_Module:ESP32-WROVER-E
Connections:
- net VBUS_5V: now reaches J5.5 (Pin_5)
- net VBUS_5V: now also U5.7 (Pin_7)
- net I2C_SCL: now reaches J2.1 (Pin_1)
- net I2C_SCL: now also R2.1, U1.8 (Pin_8), U3.5 (Pin_5)
- net GND: now reaches J2.2 (Pin_2)
- net GND: now also C1.1, C2.1, D1.1 (K), U1.37 (Pin_37), C3.1, C4.1, C5.1, U2.18 (Pin_18), U3.6 (Pin_6), U4.4 (Pin_4), U5.4 (Pin_4), U6.3 (Pin_3), U7.3 (Pin_3)
- net +3V3_DIG: now reaches J2.3 (Pin_3)
- net +3V3_DIG: now also C1.2, C2.2, R2.2, R3.2, U1.38 (Pin_38), C5.2, J4.1 (Pin_1), U2.17 (Pin_17), U3.7 (Pin_7), U6.4 (Pin_4)
- net I2C_SDA: now reaches R3.1
- net I2C_SDA: now also U1.6 (Pin_6), U3.4 (Pin_4)
- net AUD_IN: now reaches U1.24 (Pin_24)
- net AUD_IN: now also U7.7 (Pin_7)
- net UART_RX_DBG: now reaches U1.28 (Pin_28)
- net UART_RX_DBG: now also J4.4 (Pin_4)
- net UART_TX_DBG: now reaches U1.30 (Pin_30)
- net UART_TX_DBG: now also J4.5 (Pin_5)
- net LED_STAT: now reaches U1.32 (Pin_32)
- net LED_STAT: now also R1.2
- net EN: now reaches U1.34 (Pin_34)
- net EN: now also J4.3 (Pin_3)
- net IO0: now reaches U1.36 (Pin_36)
- net IO0: now also J4.2 (Pin_2)
- net VBAT_RAW: now reaches J1.1 (Pin_1)
- net VBAT_RAW: now also U5.6 (Pin_6)
- net SPK_OUT_P: now reaches J3.1 (Pin_1)
- net SPK_OUT_P: now also U7.6 (Pin_6)
- net LED_A: now reaches D1.2 (A)
- net LED_A: now also R1.1
- new net +3V3_AUD: C4.2, U4.5 (Pin_5), U7.4 (Pin_4)
- new net CAM_D0: U2.9 (Pin_9)
- new net CAM_D1: U2.10 (Pin_10)
- new net CAM_D2: U2.7 (Pin_7)
- new net CAM_D3: U2.8 (Pin_8)
- new net CAM_D4: U2.5 (Pin_5)
- new net CAM_D5: U2.6 (Pin_6)
- new net CAM_D6: U2.3 (Pin_3)
- new net CAM_D7: U2.4 (Pin_4)
- new net CAM_HREF: U2.12 (Pin_12)
- new net CAM_PCLK: U2.14 (Pin_14)
- new net CAM_SIOC: U2.15 (Pin_15)
- new net CAM_SIOD: U2.16 (Pin_16)
- new net CAM_VSYNC: U2.11 (Pin_11)
- new net CAM_XCLK: U2.13 (Pin_13)
- new net I2S_BCLK: U4.3 (Pin_3)
- new net I2S_SD_IN: U4.1 (Pin_1)
- new net I2S_WS: U4.2 (Pin_2)
- new net SPK_OUT_N: U7.5 (Pin_5)
- new net VSYS: C3.2, U5.5 (Pin_5), U6.5 (Pin_5)

Commit message: kicad source of truth
Parts:
- removed J1: BATTERY_1S, Connector_JST:JST_PH_B2B-PH-K_1x02_P2.00mm_Vertical, symbol Connector_Generic:Conn_01x02
- removed J2: OLED_I2C_PANEL, Connector_PinHeader_2.54mm:PinHeader_1x04_P2.54mm_Vertical, symbol Connector_Generic:Conn_01x04
- removed J3: SPEAKER_8OHM, Connector_PinHeader_2.54mm:PinHeader_1x02_P2.54mm_Vertical, symbol Connector_Generic:Conn_01x02
- removed J4: UART_BOOT_DEBUG, Connector_PinHeader_2.54mm:PinHeader_1x06_P2.54mm_Vertical, symbol Connector_Generic:Conn_01x06
- removed J5: USBC_POWER_IN, Connector_USB:USB_C_Receptacle_HRO_TYPE-C-31-M-12, symbol Connector_Generic:Conn_01x06
- removed U1: ESP32_WROVER_E_CORE, RF_Module:ESP32-WROVER-E, symbol Connector_Generic:Conn_02x19_Odd_Even
- removed U2: OV2640_CAMERA_IF, Connector_FFC-FPC:TE_1734839-0_1x20-1MP_P0.5mm_Horizontal, symbol Connector_Generic:Conn_02x10_Odd_Even
- removed U3: MPU6050_CORE, Package_QFN:QFN-24-1EP_4x4mm_P0.5mm_EP2.6x2.6mm, symbol Connector_Generic:Conn_01x08
- removed U4: INMP441_CORE, Package_LGA:LGA-6_3x4mm_P0.5mm, symbol Connector_Generic:Conn_01x06
- removed U6: REGULATOR_3V3_CORE, Package_TO_SOT_SMD:SOT-223-3_TabPin2, symbol Connector_Generic:Conn_01x05
- added J1: USBC_POWER_IN, Connector_USB:USB_C_Receptacle_HRO_TYPE-C-31-M-12, symbol Connector_Generic:Conn_01x06
- added J2: BATTERY_1S, Connector_JST:JST_GH_SM02B-GHS-TB_1x02-1MP_P1.25mm_Horizontal, symbol Connector_Generic:Conn_01x02
- added J3: MICRO_USB_PROG, Connector_USB:USB_Micro-B_Molex-105017-0001, symbol Connector_Generic:Conn_01x05
- added TP1: TP_I2C_SCL, TestPoint:TestPoint_Pad_D1.0mm, symbol Connector_Generic:Conn_01x01
- added TP2: TP_I2C_SDA, TestPoint:TestPoint_Pad_D1.0mm, symbol Connector_Generic:Conn_01x01
- added TP3: TP_UART_TX, TestPoint:TestPoint_Pad_D1.0mm, symbol Connector_Generic:Conn_01x01
- added TP4: TP_UART_RX, TestPoint:TestPoint_Pad_D1.0mm, symbol Connector_Generic:Conn_01x01
- added TP5: TP_EN, TestPoint:TestPoint_Pad_D1.0mm, symbol Connector_Generic:Conn_01x01
- added TP6: TP_IO0, TestPoint:TestPoint_Pad_D1.0mm, symbol Connector_Generic:Conn_01x01
- added TP7: TP_SPK_P, TestPoint:TestPoint_Pad_D1.0mm, symbol Connector_Generic:Conn_01x01
- added TP8: TP_SPK_N, TestPoint:TestPoint_Pad_D1.0mm, symbol Connector_Generic:Conn_01x01
- added U1: LIION_CHARGER_IC_CORE, Package_SO:SOIC-8_3.9x4.9mm_P1.27mm, symbol Connector_Generic:Conn_01x08
- added U2: USB_UART_BRIDGE_CORE, Package_DFN_QFN:QFN-28-1EP_5x5mm_P0.5mm_EP3.35x3.35mm, symbol Connector_Generic:Conn_01x10
- added U3: REGULATOR_3V3_CORE, Package_TO_SOT_SMD:SOT-223-3_TabPin2, symbol Connector_Generic:Conn_01x05
- added U4: ESP32_WROVER_E_CORE, RF_Module:ESP32-WROOM-32E, symbol Connector_Generic:Conn_02x19_Odd_Even
- added U6: OV2640_CAMERA_IF, Connector_FFC-FPC:TE_1734839-0_1x20-1MP_P0.5mm_Horizontal, symbol Connector_Generic:Conn_02x10_Odd_Even
- added U8: INMP441_CORE, Package_LGA:LGA-6_3x4mm_P0.5mm, symbol Connector_Generic:Conn_01x06
- C2: value 100nF -> 10uF
- C3: value 10uF -> 100nF
- R1: value 1k -> 10k
- R2: value 10k -> 1k
- U5: value LIION_CHARGER_IC_CORE -> AUDIO_AMP_CORE; footprint Package_SO:SOIC-8_3.9x4.9mm_P1.27mm -> Package_SO:SOIC-16_3.9x9.9mm_P1.27mm
- U7: value AUDIO_AMP_CORE -> MPU6050_CORE; footprint Package_SO:SOIC-16_3.9x9.9mm_P1.27mm -> Package_DFN_QFN:QFN-24-1EP_4x4mm_P0.5mm_EP2.65x2.65mm
- renumbered _TEMPLATE_C to _TEMPLATE_C1, _TEMPLATE_D to _TEMPLATE_D1, _TEMPLATE_R to _TEMPLATE_R1
Connections:
- net +3V3_AUD: now also C5.2, U5.4 (Pin_4), U8.5 (Pin_5); no longer C4.2, U7.4 (Pin_4)
- net +3V3_DIG: now also C3.2, C4.2, R1.2, R4.2, R5.2, U7.7 (Pin_7), U2.1 (Pin_1), U3.4 (Pin_4), U4.38 (Pin_38), U6.17 (Pin_17); no longer C1.2, C5.2, R2.2
- net AUD_IN: now also U5.7 (Pin_7), U4.24 (Pin_24); no longer U7.7 (Pin_7)
- net CAM_D0: now also U6.9 (Pin_9)
- net CAM_D1: now also U6.10 (Pin_10)
- net CAM_D2: now also U6.7 (Pin_7)
- net CAM_D3: now also U6.8 (Pin_8)
- net CAM_D4: now also U6.5 (Pin_5)
- net CAM_D5: now also U6.6 (Pin_6)
- net CAM_D6: now also U6.3 (Pin_3)
- net CAM_D7: now also U6.4 (Pin_4)
- net CAM_HREF: now also U6.12 (Pin_12)
- net CAM_PCLK: now also U6.14 (Pin_14)
- net CAM_SIOC: now also U6.15 (Pin_15)
- net CAM_SIOD: now also U6.16 (Pin_16)
- net CAM_VSYNC: now also U6.11 (Pin_11)
- net CAM_XCLK: now also U6.13 (Pin_13)
- net EN: now also R4.1, TP5.1 (Pin_1), U2.3 (Pin_3), U4.34 (Pin_34)
- net GND: now also U5.3 (Pin_3), U7.6 (Pin_6), J3.1 (Pin_1), U1.4 (Pin_4), U2.8 (Pin_8), U3.3 (Pin_3), U4.37 (Pin_37), U6.18 (Pin_18), U8.4 (Pin_4); no longer U5.4 (Pin_4), U7.3 (Pin_3)
- net I2C_SCL: now also R1.1, U7.5 (Pin_5), TP1.1 (Pin_1), U4.8 (Pin_8); no longer R2.1
- net I2C_SDA: now also U7.4 (Pin_4), TP2.1 (Pin_1), U4.6 (Pin_6)
- net I2S_BCLK: now also U8.3 (Pin_3)
- net I2S_SD_IN: now also U8.1 (Pin_1)
- net I2S_WS: now also U8.2 (Pin_2)
- net IO0: now also R5.1, TP6.1 (Pin_1), U2.2 (Pin_2), U4.36 (Pin_36)
- net LED_A: now also R2.1; no longer R1.1
- net LED_STAT: now also R2.2, U4.32 (Pin_32); no longer R1.2
- net SPK_OUT_N: now also U5.5 (Pin_5), TP8.1 (Pin_1); no longer U7.5 (Pin_5)
- net SPK_OUT_P: now also U5.6 (Pin_6), TP7.1 (Pin_1); no longer U7.6 (Pin_6)
- net UART_RX_DBG: now also TP4.1 (Pin_1), U2.5 (Pin_5), U4.28 (Pin_28)
- net UART_TX_DBG: now also TP3.1 (Pin_1), U2.4 (Pin_4), U4.30 (Pin_30)
- net VBAT_RAW: now also J2.1 (Pin_1), U1.6 (Pin_6); no longer U5.6 (Pin_6)
- net VBUS_5V: now also J1.5 (Pin_5), J3.5 (Pin_5), U1.7 (Pin_7), U2.9 (Pin_9); no longer U5.7 (Pin_7)
- net VSYS: now also C1.2, U1.5 (Pin_5), U3.5 (Pin_5); no longer C3.2, U5.5 (Pin_5)
- new net USB_PROG_D+: J3.3 (Pin_3), U2.7 (Pin_7)
- new net USB_PROG_D-: J3.4 (Pin_4), U2.6 (Pin_6)
