File: Hardware/Frame/espglasses/espglasses.kicad_pcb (KiCad board)
At the start: 2 copper layers, 170 x 45 mm, 13 parts, among them J1 BATTERY_1S, J2 OLED_SH1106_I2C, J3 TOUCH_INPUTS, J4 AUDIO_OUT_MONO, J5 UART_BOOT_DEBUG, J6 LED_STATUS, U1 ESP32_DEV_BOARD_PIN_BREAKOUT

Commit message: kicad checkpoint 2
Parts:
- removed J6: LED_STATUS, PinHeader_1x02_P2.54mm_Vertical
- added C3: 10uF, C_0603_1608Metric, F.Cu at (34.0, 32.0)
- added C4: 100nF, C_0603_1608Metric, F.Cu at (95.0, 32.0)
- added C5: 100nF, C_0603_1608Metric, F.Cu at (112.0, 32.0)
- added R4: 10k, R_0603_1608Metric, F.Cu at (120.0, 34.0)
- added R5: 10k, R_0603_1608Metric, F.Cu at (125.0, 23.0)
- added U2: OV2640_CAMERA_IF, Amphenol_F32Q-1A7x1-11020_1x20-1MP_P0.5mm_Horizontal, F.Cu at (166.0, 24.0)
- added U3: MPU6050_CORE, QFN-24-1EP_4x4mm_P0.5mm_EP2.65x2.65mm, F.Cu at (118.0, 26.0)
- added U4: INMP441_CORE, DFN-6-1EP_3x2mm_P0.5mm_EP1.65x1.35mm, F.Cu at (110.0, 26.0)
- added U5: LIION_CHARGER_IC_CORE, SOIC-8_3.9x4.9mm_P1.27mm, F.Cu at (30.0, 26.0)
- added U6: REGULATOR_3V3_CORE, SOT-223-3_TabPin2, F.Cu at (44.0, 26.0)
- added U7: AUDIO_AMP_CORE, SOIC-16_3.9x9.9mm_P1.27mm, F.Cu at (88.0, 26.0)
- J2: value OLED_SH1106_I2C -> OLED_I2C_PANEL
- J3: value TOUCH_INPUTS -> SPEAKER_8OHM
- J4: value AUDIO_OUT_MONO -> UART_BOOT_DEBUG; footprint PinHeader_1x02_P2.54mm_Vertical -> PinHeader_1x06_P2.54mm_Vertical
- J5: value UART_BOOT_DEBUG -> USBC_POWER_IN; footprint PinHeader_1x06_P2.54mm_Vertical -> USB_C_Receptacle_HRO_TYPE-C-31-M-12
- U1: value ESP32_DEV_BOARD_PIN_BREAKOUT -> ESP32_WROVER_E_CORE
- moved J5 78.5 mm to (8.00, 25.0), turned to -90 degrees
- moved C1 71.1 mm to (47.0, 32.0)
- moved C2 71.1 mm to (51.0, 32.0)
- moved J3 54.6 mm to (102.0, 42.0)
- moved J2 40.8 mm to (70.0, 42.0)
- moved D1 17.3 mm to (113.0, 37.0)
- moved R2 14.6 mm to (74.0, 34.0), turned to 90 degrees
- moved R3 14.6 mm to (78.0, 34.0), turned to 90 degrees
- moved J4 14.4 mm to (54.0, 42.0)
- moved R1 14.3 mm to (109.0, 34.0)
- moved U1 9.85 mm to (145.0, 26.0)
- moved J1 8.49 mm to (18.0, 40.0)
Connections:
- C1 pad 1: +3V3_DIG -> (no net)
- C1 pad 2: GND -> (no net)
- C2 pad 1: +3V3_DIG -> (no net)
- C2 pad 2: GND -> (no net)
- D1 pad 1: GND -> (no net)
- D1 pad 2: LED_A -> (no net)
- J1 pad 1: VBAT_RAW -> (no net)
- J1 pad 2: GND -> (no net)
- J2 pad 1: +3V3_DIG -> (no net)
- J2 pad 2: GND -> (no net)
- J2 pad 3: I2C_SCL -> (no net)
- J2 pad 4: I2C_SDA -> (no net)
- J3 pad 1: TOUCH1_IN -> (no net)
- J3 pad 2: TOUCH2_IN -> (no net)
- J4 pad 1: DAC_SUM -> (no net)
- J4 pad 2: GND -> (no net)
- R1 pad 1: LED_STAT -> (no net)
- R1 pad 2: LED_A -> (no net)
- R2 pad 1: DAC_L_OUT -> (no net)
- R2 pad 2: DAC_SUM -> (no net)
- R3 pad 1: DAC_R_OUT -> (no net)
- R3 pad 2: DAC_SUM -> (no net)
- U1 pad 1: GND -> (no net)
- U1 pad 10: UART_TX_DBG -> (no net)
- U1 pad 12: UART_RX_DBG -> (no net)
- U1 pad 14: DAC_R_OUT -> (no net)
- U1 pad 16: DAC_L_OUT -> (no net)
- U1 pad 2: +3V3_DIG -> (no net)
- U1 pad 24: TOUCH2_IN -> (no net)
- U1 pad 26: TOUCH1_IN -> (no net)
- U1 pad 32: I2C_SCL -> (no net)
- U1 pad 34: I2C_SDA -> (no net)
- U1 pad 4: IO0 -> (no net)
- U1 pad 6: EN -> (no net)
- U1 pad 8: LED_STAT -> (no net)
Other:
- board size 170 x 45 mm -> 180 x 50 mm

Commit message: kicad source of truth
Parts:
- removed J2: OLED_I2C_PANEL, PinHeader_1x04_P2.54mm_Vertical
- removed J3: SPEAKER_8OHM, PinHeader_1x02_P2.54mm_Vertical
- removed J4: UART_BOOT_DEBUG, PinHeader_1x06_P2.54mm_Vertical
- added J6: MICRO_USB_PROG, USB_Micro-B_Molex-105017-0001, F.Cu at (20.0, 25.0)
- added TP1: TP_UART_TX, TestPoint_Pad_D1.0mm, F.Cu at (54.0, 41.0)
- added TP2: TP_UART_RX, TestPoint_Pad_D1.0mm, F.Cu at (58.0, 41.0)
- added TP3: TP_EN, TestPoint_Pad_D1.0mm, F.Cu at (62.0, 41.0)
- added TP4: TP_IO0, TestPoint_Pad_D1.0mm, F.Cu at (66.0, 41.0)
- added TP5: TP_I2C_SCL, TestPoint_Pad_D1.0mm, F.Cu at (74.0, 41.0)
- added TP6: TP_I2C_SDA, TestPoint_Pad_D1.0mm, F.Cu at (78.0, 41.0)
- added TP7: TP_SPK_P, TestPoint_Pad_D1.0mm, F.Cu at (102.0, 41.0)
- added TP8: TP_SPK_N, TestPoint_Pad_D1.0mm, F.Cu at (106.0, 41.0)
- added U8: USB_UART_BRIDGE_CORE, QFN-28-1EP_5x5mm_P0.5mm_EP3.35x3.35mm, F.Cu at (70.0, 25.0)
- J1: footprint JST_PH_B2B-PH-K_1x02_P2.00mm_Vertical -> JST_GH_SM02B-GHS-TB_1x02-1MP_P1.25mm_Horizontal
- U1: footprint ESP32-WROOM-32 -> ESP32-WROOM-32E
- U2: footprint Amphenol_F32Q-1A7x1-11020_1x20-1MP_P0.5mm_Horizontal -> TE_2-1734839-0_1x20-1MP_P0.5mm_Horizontal
- moved U2 126.8 mm to (40.0, 10.0), turned to 0 degrees
- moved R4 26.0 mm to (121.0, 8.00)
- moved C5 17.9 mm to (104.0, 16.0)
- moved U3 17.2 mm to (108.0, 12.0)
- moved R5 15.0 mm to (125.0, 8.00)
- moved U1 12.0 mm to (145.0, 38.0)
- moved U4 10.6 mm to (117.0, 18.0)
- moved U7 4.12 mm to (92.0, 25.0)
- moved D1 3.00 mm to (113.0, 34.0)
- moved U6 2.24 mm to (46.0, 25.0)
- moved C1 1.41 mm to (46.0, 33.0)
- moved C2 1.41 mm to (50.0, 33.0)
- moved U5 1.41 mm to (31.0, 25.0)
- moved C3 1.00 mm to (34.0, 33.0)
- moved C4 1.00 mm to (95.0, 33.0)
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
Commit message: ide crashed mid response...
Connections:
- C1 pad 1: (no net) -> +3V3_DIG
- C1 pad 2: (no net) -> GND
- C2 pad 1: (no net) -> +3V3_DIG
- C2 pad 2: (no net) -> GND
- C3 pad 1: (no net) -> VSYS
- C3 pad 2: (no net) -> GND
- D1 pad 1: (no net) -> GND
- D1 pad 2: (no net) -> LED_A
- J1 pad 1: (no net) -> VBAT_RAW
- J1 pad 2: (no net) -> GND
- J6 pad 1: (no net) -> VBUS_5V
- J6 pad 2: (no net) -> USB_PROG_D-
- J6 pad 3: (no net) -> USB_PROG_D+
- J6 pad 5: (no net) -> GND
- J6 pad 6: (no net) -> GND
- R1 pad 1: (no net) -> LED_STAT
- R1 pad 2: (no net) -> LED_A
- R2 pad 1: (no net) -> +3V3_DIG
- R2 pad 2: (no net) -> I2C_SCL
- R3 pad 1: (no net) -> +3V3_DIG
- R3 pad 2: (no net) -> I2C_SDA
- R4 pad 1: (no net) -> +3V3_DIG
- R4 pad 2: (no net) -> EN
- R5 pad 1: (no net) -> +3V3_DIG
- R5 pad 2: (no net) -> IO0
- TP1 pad 1: (no net) -> UART_TX_DBG
- TP2 pad 1: (no net) -> UART_RX_DBG
- TP3 pad 1: (no net) -> EN
- TP4 pad 1: (no net) -> IO0
- TP5 pad 1: (no net) -> I2C_SCL
- TP6 pad 1: (no net) -> I2C_SDA
- U1 pad 1: (no net) -> GND
- U1 pad 10: (no net) -> UART_TX_DBG
- U1 pad 12: (no net) -> UART_RX_DBG
- U1 pad 2: (no net) -> +3V3_DIG
- U1 pad 32: (no net) -> I2C_SCL
- U1 pad 34: (no net) -> I2C_SDA
- U1 pad 4: (no net) -> IO0
- U1 pad 6: (no net) -> EN
- U1 pad 8: (no net) -> LED_STAT
- U5 pad 1: (no net) -> VBUS_5V
- U5 pad 2: (no net) -> VBAT_RAW
- U5 pad 3: (no net) -> VSYS
- U5 pad 4: (no net) -> GND
- U6 pad 1: (no net) -> VSYS
- U6 pad 2: (no net) -> +3V3_DIG
- U6 pad 3: (no net) -> GND
- U8 pad 1: (no net) -> VBUS_5V
- U8 pad 10: (no net) -> GND
- U8 pad 2: (no net) -> GND
- U8 pad 3: (no net) -> USB_PROG_D+
- U8 pad 4: (no net) -> USB_PROG_D-
- U8 pad 5: (no net) -> UART_RX_DBG
- U8 pad 6: (no net) -> UART_TX_DBG
- U8 pad 7: (no net) -> EN
- U8 pad 8: (no net) -> IO0
- U8 pad 9: (no net) -> +3V3_DIG
Routing:
- net LED_STAT: track 0.00 -> 29.1 mm
- net +3V3_DIG: track 0.00 -> 18.6 mm
- net VSYS: track 0.00 -> 8.74 mm
- net I2C_SDA: track 0.00 -> 7.83 mm
- net I2C_SCL: track 0.00 -> 7.83 mm
- net LED_A: track 0.00 -> 3.96 mm
Changed lines of the file:
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@@
 	(net 1 "GND")
 	(net 2 "VBUS_5V")
+	(net 3 "USB_PROG_D-")
+	(net 4 "USB_PROG_D+")
+	(net 5 "VBAT_RAW")
+	(net 6 "VSYS")
+	(net 7 "+3V3_DIG")
+	(net 8 "IO0")
+	(net 9 "EN")
+	(net 10 "LED_STAT")
+	(net 11 "UART_TX_DBG")
+	(net 12 "UART_RX_DBG")
+	(net 13 "I2C_SCL")
+	(net 14 "I2C_SDA")
+	(net 15 "LED_A")
 	(footprint "TestPoint_Pad_D1.0mm"
 		(layer "F.Cu")
@@
 			(size 1 1)
 			(layers "F.Cu" "F.Mask")
+			(net 8 "IO0")
 		)
 		(embedded_fonts no)
@@
 			(layers "F.Cu" "F.Mask" "F.Paste")
 			(roundrect_rratio 0.25)
+			(net 6 "VSYS")
 		)
 		(pad "2" smd roundrect
@@
 			(layers "F.Cu" "F.Mask" "F.Paste")
 			(roundrect_rratio 0.25)
+			(net 1 "GND")
 		)
 		(embedded_fonts no)
@@
 			(layers "F.Cu" "F.Mask" "F.Paste")
 			(roundrect_rratio 0.25)
+			(net 10 "LED_STAT")
 		)
 		(pad "2" smd roundrect
@@
 			(layers "F.Cu" "F.Mask" "F.Paste")
 			(roundrect_rratio 0.25)
+			(net 15 "LED_A")
 		)
 		(embedded_fonts no)
@@
 			(layers "F.Cu" "F.Mask" "F.Paste")
 			(roundrect_rratio 0.25)
+			(net 2 "VBUS_5V")
 		)
 		(pad "2" smd roundrect
@@
 			(layers "F.Cu" "F.Mask" "F.Paste")
 			(roundrect_rratio 0.25)
+			(net 5 "VBAT_RAW")
 		)
 		(pad "3" smd roundrect
@@
 			(layers "F.Cu" "F.Mask" "F.Paste")
 			(roundrect_rratio 0.25)
+			(net 6 "VSYS")
 		)
 		(pad "4" smd roundrect
@@
 			(layers "F.Cu" "F.Mask" "F.Paste")
 			(roundrect_rratio 0.25)
+			(net 1 "GND")
 		)
 		(pad "5" smd roundrect
@@
 			(size 1 1)
 			(layers "F.Cu" "F.Mask")
+			(net 12 "UART_RX_DBG")
 		)
 		(embedded_fonts no)
@@
 			(layers "F.Cu" "F.Mask" "F.Paste")
 			(roundrect_rratio 0.25)
+			(net 7 "+3V3_DIG")
 		)
 		(pad "2" smd roundrect
@@
 			(layers "F.Cu" "F.Mask" "F.Paste")
 			(roundrect_rratio 0.25)
+			(net 13 "I2C_SCL")
 		)
 		(embedded_fonts no)
@@
 			(layers "F.Cu" "F.Mask" "F.Paste")
 			(roundrect_rratio 0.25)
+			(net 2 "VBUS_5V")
 		)
 		(pad "2" smd roundrect
@@
 			(layers "F.Cu" "F.Mask" "F.Paste")
 			(roundrect_rratio 0.25)
+			(net 1 "GND")
 		)
 		(pad "3" smd roundrect
@@
 			(layers "F.Cu" "F.Mask" "F.Paste")
 			(roundrect_rratio 0.25)
+			(net 4 "USB_PROG_D+")
 		)
 		(pad "4" smd roundrect
@@
 			(layers "F.Cu" "F.Mask" "F.Paste")
 			(roundrect_rratio 0.25)
+			(net 3 "USB_PROG_D-")
 		)
 		(pad "5" smd roundrect
@@
 			(layers "F.Cu" "F.Mask" "F.Paste")
 			(roundrect_rratio 0.25)
+			(net 12 "UART_RX_DBG")
 		)
 		(pad "6" smd roundrect
@@
 			(layers "F.Cu" "F.Mask" "F.Paste")
 			(roundrect_rratio 0.25)
+			(net 11 "UART_TX_DBG")
 		)
 		(pad "7" smd roundrect
@@
 			(layers "F.Cu" "F.Mask" "F.Paste")
 			(roundrect_rratio 0.25)
+			(net 9 "EN")
 		)
 		(pad "8" smd roundrect
@@
 			(layers "F.Cu" "F.Mask" "F.Paste")
 			(roundrect_rratio 0.25)
+			(net 8 "IO0")
 		)
 		(pad "9" smd roundrect
@@
 			(layers "F.Cu" "F.Mask" "F.Paste")
 			(roundrect_rratio 0.25)
+			(net 7 "+3V3_DIG")
 		)
 		(pad "10" smd roundrect
@@
 			(layers "F.Cu" "F.Mask" "F.Paste")
 			(roundrect_rratio 0.25)
+			(net 1 "GND")
 		)
 		(pad "11" smd roundrect
@@
 			(size 1 1)
 			(layers "F.Cu" "F.Mask")
+			(net 14 "I2C_SDA")
 		)
 		(embedded_fonts no)
@@
 			(size 1 1)
 			(layers "F.Cu" "F.Mask")
+			(net 11 "UART_TX_DBG")
 		)
 		(embedded_fonts no)
@@
 			(layers "F.Cu" "F.Mask" "F.Paste")
 			(roundrect_rratio 0.25)
+			(net 1 "GND")
 		)
 		(pad "2" smd roundrect
@@
 			(layers "F.Cu" "F.Mask" "F.Paste")
 			(roundrect_rratio 0.25)
+			(net 15 "LED_A")
 		)
 		(embedded_fonts no)
@@
 			(size 1 1)
 			(layers "F.Cu" "F.Mask")
+			(net 9 "EN")
 		)
 		(embedded_fonts no)
@@
 			(layers "F.Cu" "F.Mask" "F.Paste")
 			(roundrect_rratio 0.25)
+			(net 7 "+3V3_DIG")
 		)
 		(pad "2" smd roundrect
@@
 			(layers "F.Cu" "F.Mask" "F.Paste")
 			(roundrect_rratio 0.25)
+			(net 1 "GND")
 		)
 		(embedded_fonts no)
@@
 			(size 1.5 0.9)
 			(layers "F.Cu" "F.Mask" "F.Paste")
+			(net 1 "GND")
 		)
 		(pad "2" smd rect
@@
 			(size 1.5 0.9)
 			(layers "F.Cu" "F.Mask" "F.Paste")
+			(net 7 "+3V3_DIG")
 		)
 		(pad "3" smd rect
@@
 			(size 1.5 0.9)
 			(layers "F.Cu" "F.Mask" "F.Paste")
+			(net 8 "IO0")
 		)
 		(pad "5" smd rect
@@
 			(size 1.5 0.9)
 			(layers "F.Cu" "F.Mask" "F.Paste")
+			(net 9 "EN")
 		)
 		(pad "7" smd rect
@@
 			(size 1.5 0.9)
 			(layers "F.Cu" "F.Mask" "F.Paste")
+			(net 10 "LED_STAT")
 		)
 		(pad "9" smd rect
@@
 			(size 1.5 0.9)
 			(layers "F.Cu" "F.Mask" "F.Paste")
+			(net 11 "UART_TX_DBG")
 		)
 		(pad "11" smd rect
@@
 			(size 1.5 0.9)
 			(layers "F.Cu" "F.Mask" "F.Paste")
+			(net 12 "UART_RX_DBG")
 		)
 		(pad "13" smd rect
@@
 			(size 1.5 0.9)
 			(layers "F.Cu" "F.Mask" "F.Paste")
+			(net 13 "I2C_SCL")
 		)
 		(pad "33" smd rect
@@
 			(size 1.5 0.9)
 			(layers "F.Cu" "F.Mask" "F.Paste")
+			(net 14 "I2C_SDA")
 		)
 		(pad "35" smd rect
@@
 			(layers "F.Cu" "F.Mask" "F.Paste")
 			(roundrect_rratio 0.25)
+			(net 7 "+3V3_DIG")
 		)
 		(pad "2" smd roundrect
@@
 			(layers "F.Cu" "F.Mask" "F.Paste")
 			(roundrect_rratio 0.25)
+			(net 9 "EN")
 		)
 		(embedded_fonts no)
@@
 			(layers "F.Cu" "F.Mask" "F.Paste")
 			(roundrect_rratio 0.25)
+			(net 7 "+3V3_DIG")
 		)
 		(pad "2" smd roundrect
@@
 			(layers "F.Cu" "F.Mask" "F.Paste")
 			(roundrect_rratio 0.25)
+			(net 8 "IO0")
 		)
 		(embedded_fonts no)
@@
 			(size 0.4 1.35)
 			(layers "F.Cu" "F.Mask" "F.Paste")
+			(net 2 "VBUS_5V")
 		)
 		(pad "2" smd rect
@@
 			(size 0.4 1.35)
 			(layers "F.Cu" "F.Mask" "F.Paste")
+			(net 3 "USB_PROG_D-")
 		)
 		(pad "3" smd rect
@@
 			(size 0.4 1.35)
 			(layers "F.Cu" "F.Mask" "F.Paste")
+			(net 4 "USB_PROG_D+")
 		)
 		(pad "4" smd rect
@@
 			(size 0.4 1.35)
 			(layers "F.Cu" "F.Mask" "F.Paste")
+			(net 1 "GND")
 		)
 		(pad "6" thru_hole oval
@@
 			(layers "*.Cu" "*.Mask")
 			(remove_unused_layers no)
+			(net 1 "GND")
 		)
 		(pad "6" smd rect
@@
 			(size 1.2 1.9)
 			(layers "F.Cu" "F.Mask")
+			(net 1 "GND")
 		)
 		(pad "6" thru_hole circle
@@
 			(layers "*.Cu" "*.Mask")
 			(remove_unused_layers no)
+			(net 1 "GND")
 		)
 		(pad "6" smd rect
@@
 			(size 1.5 1.9)
 			(layers "F.Cu" "F.Mask" "F.Paste")
+			(net 1 "GND")
 		)
 		(pad "6" smd rect
@@
 			(size 1.5 1.9)
 			(layers "F.Cu" "F.Mask" "F.Paste")
+			(net 1 "GND")
 		)
 		(pad "6" thru_hole circle
@@
 			(layers "*.Cu" "*.Mask")
 			(remove_unused_layers no)
+			(net 1 "GND")
 		)
 		(pad "6" smd rect
@@
 			(size 1.2 1.9)
 			(layers "F.Cu" "F.Mask")
+			(net 1 "GND")
 		)
 		(pad "6" thru_hole oval
@@
 			(layers "*.Cu" "*.Mask")
 			(remove_unused_layers no)
+			(net 1 "GND")
 		)
 		(embedded_fonts no)
@@
 			(layers "F.Cu" "F.Mask" "F.Paste")
 			(roundrect_rratio 0.25)
+			(net 5 "VBAT_RAW")
 		)
 		(pad "2" smd roundrect
@@
 			(layers "F.Cu" "F.Mask" "F.Paste")
 			(roundrect_rratio 0.25)
+			(net 1 "GND")
 		)
 		(pad "MP" smd roundrect
@@
 			(size 1 1)
 			(layers "F.Cu" "F.Mask")
+			(net 13 "I2C_SCL")
 		)
 		(embedded_fonts no)
@@
 			(layers "F.Cu" "F.Mask" "F.Paste")
 			(roundrect_rratio 0.25)
+			(net 7 "+3V3_DIG")
 		)
 		(pad "2" smd roundrect
@@
 			(layers "F.Cu" "F.Mask" "F.Paste")
 			(roundrect_rratio 0.25)
+			(net 14 "I2C_SDA")
 		)
 		(embedded_fonts no)
@@
 			(layers "F.Cu" "F.Mask" "F.Paste")
 			(roundrect_rratio 0.25)
+			(net 7 "+3V3_DIG")
 		)
 		(pad "2" smd roundrect
@@
 			(layers "F.Cu" "F.Mask" "F.Paste")
 			(roundrect_rratio 0.25)
+			(net 1 "GND")
 		)
 		(embedded_fonts no)
@@
 			(layers "F.Cu" "F.Mask" "F.Paste")
 			(roundrect_rratio 0.25)
+			(net 6 "VSYS")
 		)
 		(pad "2" smd roundrect
@@
 			(layers "F.Cu" "F.Mask" "F.Paste")
 			(roundrect_rratio 0.25)
+			(net 7 "+3V3_DIG")
 		)
 		(pad "2" smd roundrect
@@
 			(layers "F.Cu" "F.Mask" "F.Paste")
 			(roundrect_rratio 0.25)
+			(net 7 "+3V3_DIG")
 		)
 		(pad "3" smd roundrect
@@
 			(layers "F.Cu" "F.Mask" "F.Paste")
 			(roundrect_rratio 0.25)
+			(net 1 "GND")
 		)
 		(embedded_fonts no)
@@
 		(layer "Edge.Cuts")
 	)
+	(segment
+		(start 28.525 25.635)
+		(end 33.225 33)
+		(width 0.3)
+		(layer "F.Cu")
+		(net 6)
+	)
+	(segment
+		(start 42.85 25)
+		(end 49.225 33)
+		(width 0.3)
+		(layer "F.Cu")
+		(net 7)
+	)
+	(segment
+		(start 42.85 25)
+		(end 45.225 33)
+		(width 0.3)
+		(layer "F.Cu")
+		(net 7)
+	)
+	(segment
+		(start 136.25 41.63)
+		(end 108.175 34)
+		(width 0.25)
+		(layer "F.Cu")
+		(net 10)
+	)
+	(segment
+		(start 74 33.174999)
+		(end 74 41)
+		(width 0.25)
+		(layer "F.Cu")
+		(net 13)
+	)
+	(segment
+		(start 78 33.174999)
+		(end 78 41)
+		(width 0.25)
+		(layer "F.Cu")
+		(net 14)
+	)
+	(segment
+		(start 109.825 34)
+		(end 113.7875 34)
+		(width 0.25)
+		(layer "F.Cu")
+		(net 15)
+	)
 	(embedded_fonts no)

Commit message: refactor
Routing:
- net LED_STAT: track 29.1 -> 0.00 mm
- net I2C_SDA: track 7.83 -> 0.00 mm
- net I2C_SCL: track 7.83 -> 0.00 mm
- net +3V3_DIG: track 18.6 -> 24.8 mm
- net LED_A: track 3.96 -> 0.00 mm
- net VSYS: track 8.74 -> 12.1 mm
Changed lines of the file:
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@@
 	)
 	(segment
-		(start 28.525 25.635)
+		(start 31 25.635)
+		(end 31 33)
+		(width 0.3)
+		(layer "F.Cu")
+		(net 6)
+	)
+	(segment
+		(start 31 33)
 		(end 33.225 33)
 		(width 0.3)
@@
 	)
 	(segment
-		(start 42.85 25)
+		(start 28.525 25.635)
+		(end 31 25.635)
+		(width 0.3)
+		(layer "F.Cu")
+		(net 6)
+	)
+	(segment
+		(start 49.225 25)
 		(end 49.225 33)
 		(width 0.3)
@@
 	(segment
 		(start 42.85 25)
+		(end 45.225 25)
+		(width 0.3)
+		(layer "F.Cu")
+		(net 7)
+	)
+	(segment
+		(start 45.225 25)
 		(end 45.225 33)
 		(width 0.3)
@@
 	)
 	(segment
-		(start 136.25 41.63)
-		(end 108.175 34)
-		(width 0.25)
+		(start 42.85 25)
+		(end 49.225 25)
+		(width 0.3)
 		(layer "F.Cu")
-		(net 10)
-	)
-	(segment
-		(start 74 33.174999)
-		(end 74 41)
-		(width 0.25)
-		(layer "F.Cu")
-		(net 13)
-	)
-	(segment
-		(start 78 33.174999)
-		(end 78 41)
-		(width 0.25)
-		(layer "F.Cu")
-		(net 14)
-	)
-	(segment
-		(start 109.825 34)
-		(end 113.7875 34)
-		(width 0.25)
-		(layer "F.Cu")
-		(net 15)
+		(net 7)
 	)
 	(embedded_fonts no)
