File: Hardware/KiCAD_Rebuild_2026_04_08/smart_glasses_rebuild_clean.kicad_pcb (KiCad board)
At the start: 2 copper layers, 0 parts

Commit message: kicad manual checkpoint
Other:
- board outline added: 150 x 50 mm
Changed lines of the file:
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@@
 	)
 	(paper "A4")
+	(title_block
+		(title "smart_glasses_rebuild_clean")
+		(date "2026-04-11")
+	)
 	(layers
 		(0 "F.Cu" signal)
@@
 	)
 	(net 0 "")
+	(gr_rect
+		(start 66.85 31.1)
+		(end 216.85 81.1)
+		(stroke
+			(width 0.05)
+			(type default)
+		)
+		(fill no)
+		(layer "Edge.Cuts")
+	)
 	(embedded_fonts no)
 )
